Commit message: Hello im sorry for no message

File: gazebo/rover.urdf (robot description, URDF)
Before this commit: robot rover, 12 links, 11 joints
Joints:
- joint left_front_steer_joint: type revolute -> continuous
- joint left_rear_steer_joint: type revolute -> continuous
- joint right_front_steer_joint: type revolute -> continuous
- joint right_rear_steer_joint: type revolute -> continuous
